Commit message: update

File: src/urdf/camera.xacro (robot description, xacro)
@@ -12,5 +12,5 @@
                     <cylinder length="0.05" radius="0.03"/>
                 </geometry>
-                <material name="preto"/>
+                <!-- <material name="preto"/> -->
             </visual>
             <collision>
